File: adaptadora/acp_y_arp.sch (KiCad schematic (older format))
At the start: 60 parts, among them J13 Conn_Coaxial, J14 Conn_Coaxial, J15 Conn_Coaxial, J16 Conn_Coaxial, J17 Conn_Coaxial, J18 Conn_Coaxial, J19 Conn_Coaxial, J20 Conn_Coaxial, J21 Conn_Coaxial, U10 SN74LVC2T45DCUR, U3 LM361MX_NOPB, U4 LM361MX_NOPB, U5 LM361MX_NOPB, U6 TLV2772IDR, U7 TLV2772IDR, U8 TLV2772IDR, U9 SN74LVC2T45DCUR

Commit message: correcciones implementadas
Parts:
- removed C12, C13, C14: 1uF-16V, symbol Device:CP1
- removed C20, C21, C22, C23, C24, C25, C26, C27, C28, C29, C30: 0.1uF-50V, symbol Device:C
- removed D5, D6: D_TVS, symbol Device:D_TVS
- removed J18, J19, J20, J21: Conn_Coaxial, symbol Connector:Conn_Coaxial
- removed JP10, JP7, JP8, JP9: Jumper_3_Open, symbol Jumper:Jumper_3_Open
- removed R7, R8, R9: 100 - 1/8W - 5%, symbol Device:R
- removed RV10, RV7, RV8, RV9: R_POT, symbol Device:R_POT
- removed TP3: TestPoint, symbol Connector:TestPoint
- removed U10, U9: SN74LVC2T45DCUR, Package_SO:VSSOP-8_2.4x2.1mm_P0.5mm, symbol Logic_LevelTranslator:SN74LVC2T45DCUR
- removed U3, U4, U5: LM361MX_NOPB, SOIC127P600X175-14N, symbol sincronismo-rescue:LM361MX_NOPB-LM361MX_NOPB
- removed U6, U7, U8: TLV2772IDR, SOIC127P600X175-8N, symbol TLV2772IDR:TLV2772IDR
- added C10, C11, C12, C13, C14: 0.1uF-50V, symbol Device:C
- added C8, C9: 1uF-16V, symbol Device:CP1
- added D3: D_TVS, symbol Device:D_TVS
- added J12: Conn_Coaxial, symbol Connector:Conn_Coaxial
- added JP3, JP4: Jumper_3_Open, symbol Jumper:Jumper_3_Open
- added R3: 50 - 1/2W - 5%, symbol Device:R
- added RV3, RV4: R_POT, symbol Device:R_POT
- added U1_1 (x2): LM361MX_NOPB, SOIC127P600X175-14N, symbol sincronismo-rescue:LM361MX_NOPB-LM361MX_NOPB
- added U2_1 (x2): TLV2772IDR, SOIC127P600X175-8N, symbol TLV2772IDR:TLV2772IDR
- added U3_1: SN74LVC2T45DCUR, Package_SO:VSSOP-8_2.4x2.1mm_P0.5mm, symbol Logic_LevelTranslator:SN74LVC2T45DCUR
- R5, R6: value 50 - 1/2W - 5% -> 100 - 1/8W - 5%
Connections:
- net PRF is gone; now on net ACP: TP1.1
- net +12V: now also C12.1, C13.1, U1_1.1 (V+), U1_1.1 (V+); no longer C18.1, C19.1
- net +3V3: now also C19.1, U3_1.1 (VCCA)
- net +5V: now also C16.1, C17.1, C18.2, RV5.1, RV6.1, C10.2, C11.2, U1_1.13 (STROBE1), U1_1.13 (STROBE1), U1_1.14 (VCC), U1_1.14 (VCC), U1_1.8 (STROBE2), U1_1.8 (STROBE2), U2_1.8 (VDD), U2_1.8 (VDD), U3_1.8 (VCCB); no longer C15.2, C16.2, C17.2
- net -12V: now also C15.1, C14.1, U1_1.6 (V-), U1_1.6 (V-)
- net ACP: now also JP5.2 (C), U2_1.3 (1IN+), U2_1.5 (2IN+), U3_1.7 (B1); no longer TP2.1
- net ACP_3P3: now also U3_1.2 (A1)
- net ARP: now also JP6.2 (C), TP2.1, U2_1.3 (1IN+), U2_1.5 (2IN+), U3_1.6 (B2)
- net ARP_3P3: now also U3_1.3 (A2)
- net GND: now also C15.2, C16.2, C17.2, C18.1, C10.1, C11.1, C12.2, C13.2, C14.2, C8.2, C9.2, D3.2 (A2), J12.2 (Ext), R3.2, RV3.3, RV4.3, U1_1.10 (GND), U1_1.10 (GND), U2_1.4 (GND), U2_1.4 (GND), U3_1.4 (GND), U3_1.5 (DIR); no longer C15.1, C16.1, C17.1, C18.2, R5.2, R6.2
- net at RV5.2: now also C8.1, U1_1.4 (-IN); no longer D4.1 (A1)
- net at J16.1 (In): now also U2_1.1 (1OUT), U2_1.2 (1IN-)
- net at RV6.2: now also C9.1, U1_1.4 (-IN)
- net at J17.1 (In): now also U2_1.1 (1OUT), U2_1.2 (1IN-)
- net at J15.1 (In): now also U2_1.6 (2IN-), U2_1.7 (2OUT)
- net at R6.1: now also U1_1.3 (+IN)
- new net: J12.1 (In), JP3.1 (A), RV3.1
- new net: D3.1 (A1), R5.2, RV3.2
- new net: R5.1, U1_1.3 (+IN)
- new net: JP5.1 (A), U1_1.11 (OUT+)
- new net: JP5.3 (B), U1_1.9 (OUT-)
- new net: J14.1 (In), U2_1.6 (2IN-), U2_1.7 (2OUT)
- new net: JP6.1 (A), U1_1.11 (OUT+)
- new net: JP6.3 (B), U1_1.9 (OUT-)
- new net: JP3.2 (C), JP3.3 (B), R3.1
- new net: J13.1 (In), JP4.1 (A), RV4.1
- new net: JP4.2 (C), JP4.3 (B), R4.1
- new net: D4.1 (A1), R6.2, RV4.2
- no-connect marks 12 -> 8
Other:
- note added: "U1_X: Comparadores\nTensión de señal de entrada máxima 12 V\nTensión de señal de salida 5V"
- note added: "U2_X: Amplificadores operacionales\nSalidas duplicadas para otros equipos\nTensión de salida: 5V"
- note added: "U3_X: Convertidor de Niveles Lógicos\nTensión de señal de entrada 5 V\nTensión de señal de salida 3.3V"
- note removed: "PRF\nEntrada Radar"

Commit message: se agregan huellas, en progreso
Parts:
- J12, J13, J14, J15, J16, J17: footprint (none) -> Connector_Coaxial:SMA_Amphenol_901-144_Vertical
- renumbered U1_1 to U1_2, U2_1 to U2_2
Changed lines of the file:
@@
 F 0 "J12" H 628 2188 50  0000 C CNN
 F 1 "Conn_Coaxial" H 628 2097 50  0000 C CNN
-F 2 "" H 700 1950 50  0001 C CNN
+F 2 "Connector_Coaxial:SMA_Amphenol_901-144_Vertical" H 700 1950 50  0001 C CNN
 F 3 " ~" H 700 1950 50  0001 C CNN
 	1    700  1950
@@
 F 0 "J13" H 628 4888 50  0000 C CNN
 F 1 "Conn_Coaxial" H 628 4797 50  0000 C CNN
-F 2 "" H 700 4650 50  0001 C CNN
+F 2 "Connector_Coaxial:SMA_Amphenol_901-144_Vertical" H 700 4650 50  0001 C CNN
 F 3 " ~" H 700 4650 50  0001 C CNN
 	1    700  4650
@@
 	950  5800 1850 5800
 $Comp
-L sincronismo-rescue:LM361MX_NOPB-LM361MX_NOPB U1_1
+L sincronismo-rescue:LM361MX_NOPB-LM361MX_NOPB U1_2
 U 1 1 5DCAAD2F
 P 4100 5200
-F 0 "U1_1" H 4100 5870 50  0000 C CNN
+F 0 "U1_2" H 4100 5870 50  0000 C CNN
 F 1 "LM361MX_NOPB" H 4100 5779 50  0000 C CNN
 F 2 "SOIC127P600X175-14N" H 4100 5200 50  0001 L BNN
@@
 $EndComp
 $Comp
-L TLV2772IDR:TLV2772IDR U2_1
+L TLV2772IDR:TLV2772IDR U2_2
 U 1 1 5E2599A0
 P 7300 4650
-F 0 "U2_1" H 7300 5220 50  0000 C CNN
+F 0 "U2_2" H 7300 5220 50  0000 C CNN
 F 1 "TLV2772IDR" H 7300 5129 50  0000 C CNN
 F 2 "SOIC127P600X175-8N" H 7300 4650 50  0001 L BNN
@@
 F 0 "J17" H 8850 4325 50  0000 L CNN
 F 1 "Conn_Coaxial" H 8850 4234 50  0000 L CNN
-F 2 "" H 8750 4350 50  0001 C CNN
+F 2 "Connector_Coaxial:SMA_Amphenol_901-144_Vertical" H 8750 4350 50  0001 C CNN
 F 3 " ~" H 8750 4350 50  0001 C CNN
 	1    8750 4350
@@
 F 0 "J15" H 8100 4550 50  0000 L CNN
 F 1 "Conn_Coaxial" H 7850 4450 50  0000 L CNN
-F 2 "" H 8450 4650 50  0001 C CNN
+F 2 "Connector_Coaxial:SMA_Amphenol_901-144_Vertical" H 8450 4650 50  0001 C CNN
 F 3 " ~" H 8450 4650 50  0001 C CNN
 	1    8450 4650
@@
 F 0 "J16" H 8850 1925 50  0000 L CNN
 F 1 "Conn_Coaxial" H 8850 1834 50  0000 L CNN
-F 2 "" H 8750 1950 50  0001 C CNN
+F 2 "Connector_Coaxial:SMA_Amphenol_901-144_Vertical" H 8750 1950 50  0001 C CNN
 F 3 " ~" H 8750 1950 50  0001 C CNN
 	1    8750 1950
@@
 F 0 "J14" H 8100 2150 50  0000 L CNN
 F 1 "Conn_Coaxial" H 7850 2050 50  0000 L CNN
-F 2 "" H 8450 2250 50  0001 C CNN
+F 2 "Connector_Coaxial:SMA_Amphenol_901-144_Vertical" H 8450 2250 50  0001 C CNN
 F 3 " ~" H 8450 2250 50  0001 C CNN
 	1    8450 2250

Commit message: pcb work in progress
Parts:
- C10, C11, C12, C13, C14, C15, C16, C17, C18, C19: footprint (none) -> Capacitor_SMD:C_0805_2012Metric
- C8, C9: footprint (none) -> Resistor_SMD:R_1206_3216Metric
- D3, D4: footprint (none) -> Diode_THT:D_DO-15_P10.16mm_Horizontal
- JP3, JP4, JP5, JP6: footprint (none) -> Jumper:SolderJumper-3_P1.3mm_Open_Pad1.0x1.5mm_NumberLabels
- R3, R4: footprint (none) -> Resistor_THT:R_Axial_DIN0414_L11.9mm_D4.5mm_P15.24mm_Horizontal
- R5, R6: footprint (none) -> Resistor_SMD:R_0805_2012Metric
- RV3, RV4, RV5, RV6: footprint (none) -> Potentiometer_THT:Potentiometer_Bourns_3296W_Vertical
- TP1, TP2: footprint (none) -> TestPoint:TestPoint_THTPad_1.5x1.5mm_Drill0.7mm
- U11: renamed from U1_1; footprint SOIC127P600X175-14N -> Package_DIP:DIP-14_W7.62mm
- U12: renamed from U1_2; footprint SOIC127P600X175-14N -> Package_DIP:DIP-14_W7.62mm
- U21: renamed from U2_1; footprint SOIC127P600X175-8N -> Package_SO:SOIC-8_7.5x5.85mm_P1.27mm
- U22: renamed from U2_2; footprint SOIC127P600X175-8N -> Package_SO:SOIC-8_7.5x5.85mm_P1.27mm
- renumbered U3_1 to U31
Other:
- note added: "U1X: Comparadores\nTensión de señal de entrada máxima 12 V\nTensión de señal de salida 5V"
- note added: "U2X: Amplificadores operacionales\nSalidas duplicadas para otros equipos\nTensión de salida: 5V"
- note added: "U3X: Convertidor de Niveles Lógicos\nTensión de señal de entrada 5 V\nTensión de señal de salida 3.3V"
- note removed: "U1_X: Comparadores\nTensión de señal de entrada máxima 12 V\nTensión de señal de salida 5V"
- note removed: "U2_X: Amplificadores operacionales\nSalidas duplicadas para otros equipos\nTensión de salida: 5V"
- note removed: "U3_X: Convertidor de Niveles Lógicos\nTensión de señal de entrada 5 V\nTensión de señal de salida 3.3V"

Commit message: Componentes acomodados en PCB
Parts:
- U11, U12: footprint Package_DIP:DIP-14_W7.62mm -> Package_SO:SOIC-14_3.9x8.7mm_P1.27mm
- U21, U22: footprint Package_SO:SOIC-8_7.5x5.85mm_P1.27mm -> Package_SO:SOIC-8_3.9x4.9mm_P1.27mm
Changed lines of the file:
@@
 F 0 "U11" H 4100 3170 50  0000 C CNN
 F 1 "LM361MX_NOPB" H 4100 3079 50  0000 C CNN
-F 2 "Package_DIP:DIP-14_W7.62mm" H 4100 2500 50  0001 L BNN
+F 2 "Package_SO:SOIC-14_3.9x8.7mm_P1.27mm" H 4100 2500 50  0001 L BNN
 F 3 "SOIC-14 Texas Instruments" H 4100 2500 50  0001 L BNN
 F 4 "Texas Instruments" H 4100 2500 50  0001 L BNN "Fabricante"
@@
 F 0 "U21" H 7300 2820 50  0000 C CNN
 F 1 "TLV2772IDR" H 7300 2729 50  0000 C CNN
-F 2 "Package_SO:SOIC-8_7.5x5.85mm_P1.27mm" H 7300 2250 50  0001 L BNN
+F 2 "Package_SO:SOIC-8_3.9x4.9mm_P1.27mm" H 7300 2250 50  0001 L BNN
 F 3 "296-1902-1-ND" H 7300 2250 50  0001 L BNN
 F 4 "Texas Instruments" H 7300 2250 50  0001 L BNN "Fabricante"
@@
 F 0 "U12" H 4100 5870 50  0000 C CNN
 F 1 "LM361MX_NOPB" H 4100 5779 50  0000 C CNN
-F 2 "Package_DIP:DIP-14_W7.62mm" H 4100 5200 50  0001 L BNN
+F 2 "Package_SO:SOIC-14_3.9x8.7mm_P1.27mm" H 4100 5200 50  0001 L BNN
 F 3 "SOIC-14 Texas Instruments" H 4100 5200 50  0001 L BNN
 F 4 "Texas Instruments" H 4100 5200 50  0001 L BNN "Fabricante"
@@
 F 0 "U22" H 7300 5220 50  0000 C CNN
 F 1 "TLV2772IDR" H 7300 5129 50  0000 C CNN
-F 2 "Package_SO:SOIC-8_7.5x5.85mm_P1.27mm" H 7300 4650 50  0001 L BNN
+F 2 "Package_SO:SOIC-8_3.9x4.9mm_P1.27mm" H 7300 4650 50  0001 L BNN
 F 3 "296-1902-1-ND" H 7300 4650 50  0001 L BNN
 F 4 "Texas Instruments" H 7300 4650 50  0001 L BNN "Fabricante"

Commit message: correcciones y archivos agregados
Parts:
- D3, D4: footprint Diode_THT:D_DO-15_P10.16mm_Horizontal -> Diode_SMD:D_0201_0603Metric
Connections:
- net -12V: now also C14.2, C15.2; no longer C14.1, C15.1
- net GND: now also C14.1, C15.1; no longer C14.2, C15.2
Other:
- note added: "JP3\nSelección de Carga de Entrada R3\n\n"
- note added: "JP4\nSelección de Carga de Entrada R4\n\n"
- note added: "JP5\nSelección salida negada\n\n"
- note added: "JP6\nSelección salida negada\n\n"
- moved on the sheet: C12, C13, C14, C15
Changed lines of the file:
@@
 F 0 "D3" V 1954 2979 50  0000 L CNN
 F 1 "D_TVS" V 2045 2979 50  0000 L CNN
-F 2 "Diode_THT:D_DO-15_P10.16mm_Horizontal" H 2000 2900 50  0001 C CNN
+F 2 "Diode_SMD:D_0201_0603Metric" H 2000 2900 50  0001 C CNN
 F 3 "~" H 2000 2900 50  0001 C CNN
 	1    2000 2900
@@
 L power:GND #PWR021
 U 1 1 5DCAAD10
-P 2500 3100
-F 0 "#PWR021" H 2500 2850 50  0001 C CNN
-F 1 "GND" H 2505 2927 50  0000 C CNN
-F 2 "" H 2500 3100 50  0001 C CNN
-F 3 "" H 2500 3100 50  0001 C CNN
-	1    2500 3100
+P 2500 3300
+F 0 "#PWR021" H 2500 3050 50  0001 C CNN
+F 1 "GND" H 2505 3127 50  0000 C CNN
+F 2 "" H 2500 3300 50  0001 C CNN
+F 3 "" H 2500 3300 50  0001 C CNN
+	1    2500 3300
 	1    0    0    -1
 $EndComp
@@
 L Device:C C12
 U 1 1 5DB2F954
-P 3700 1150
-F 0 "C12" H 3900 1050 50  0000 R CNN
-F 1 "0.1uF-50V" H 3700 900 50  0000 L BNN
-F 2 "Capacitor_SMD:C_0805_2012Metric" H 3738 1000 50  0001 C CNN
-F 3 "~" H 3700 1150 50  0001 C CNN
-	1    3700 1150
+P 3150 1100
+F 0 "C12" H 2900 1150 50  0000 R CNN
+F 1 "0.1uF-50V" H 2600 1000 50  0000 L BNN
+F 2 "Capacitor_SMD:C_0805_2012Metric" H 3188 950 50  0001 C CNN
+F 3 "~" H 3150 1100 50  0001 C CNN
+	1    3150 1100
 	-1   0    0    -1
 $EndComp
@@
 L Device:C C14
 U 1 1 5DCAAD24
-P 4400 1150
-F 0 "C14" H 4150 1250 50  0000 L CNN
-F 1 "0.1uF-50V" H 3900 1150 50  0000 L CNN
-F 2 "Capacitor_SMD:C_0805_2012Metric" H 4438 1000 50  0001 C CNN
-F 3 "~" H 4400 1150 50  0001 C CNN
-	1    4400 1150
+P 3150 1500
+F 0 "C14" H 3400 1550 50  0000 L CNN
+F 1 "0.1uF-50V" H 3300 1400 50  0000 L CNN
+F 2 "Capacitor_SMD:C_0805_2012Metric" H 3188 1350 50  0001 C CNN
+F 3 "~" H 3150 1500 50  0001 C CNN
+	1    3150 1500
 	1    0    0    -1
 $EndComp
@@
 L power:GND #PWR032
 U 1 1 5DB594EF
-P 4100 1300
-F 0 "#PWR032" H 4100 1050 50  0001 C CNN
-F 1 "GND" H 4105 1127 50  0000 C CNN
-F 2 "" H 4100 1300 50  0001 C CNN
-F 3 "" H 4100 1300 50  0001 C CNN
-	1    4100 1300
+P 2800 1400
+F 0 "#PWR032" H 2800 1150 50  0001 C CNN
+F 1 "GND" H 2800 1250 50  0000 C CNN
+F 2 "" H 2800 1400 50  0001 C CNN
+F 3 "" H 2800 1400 50  0001 C CNN
+	1    2800 1400
 	1    0    0    -1
 $EndComp
@@
 L power:+12V #PWR030
 U 1 1 5DCAAD15
-P 3700 950
-F 0 "#PWR030" H 3700 800 50  0001 C CNN
-F 1 "+12V" H 3715 1123 50  0000 C CNN
-F 2 "" H 3700 950 50  0001 C CNN
-F 3 "" H 3700 950 50  0001 C CNN
-	1    3700 950
+P 3150 900
+F 0 "#PWR030" H 3150 750 50  0001 C CNN
+F 1 "+12V" H 3165 1073 50  0000 C CNN
+F 2 "" H 3150 900 50  0001 C CNN
+F 3 "" H 3150 900 50  0001 C CNN
+	1    3150 900
 	1    0    0    -1
 $EndComp
@@
 L power:-12V #PWR034
 U 1 1 5DCAAD16
-P 4400 950
-F 0 "#PWR034" H 4400 1050 50  0001 C CNN
-F 1 "-12V" H 4415 1123 50  0000 C CNN
-F 2 "" H 4400 950 50  0001 C CNN
-F 3 "" H 4400 950 50  0001 C CNN
-	1    4400 950
-	1    0    0    -1
-$EndComp
-Wire Wire Line
-	3700 1300 4100 1300
+P 3150 1750
+F 0 "#PWR034" H 3150 1850 50  0001 C CNN
+F 1 "-12V" H 3165 1923 50  0000 C CNN
+F 2 "" H 3150 1750 50  0001 C CNN
+F 3 "" H 3150 1750 50  0001 C CNN
+	1    3150 1750
+	-1   0    0    1
+$EndComp
 $Comp
 L power:+5V #PWR040
@@
 L power:GND #PWR041
 U 1 1 5DCAAD29
-P 6600 2750
-F 0 "#PWR041" H 6600 2500 50  0001 C CNN
-F 1 "GND" H 6605 2577 50  0000 C CNN
-F 2 "" H 6600 2750 50  0001 C CNN
-F 3 "" H 6600 2750 50  0001 C CNN
-	1    6600 2750
+P 6450 2900
+F 0 "#PWR041" H 6450 2650 50  0001 C CNN
+F 1 "GND" H 6455 2727 50  0000 C CNN
+F 2 "" H 6450 2900 50  0001 C CNN
+F 3 "" H 6450 2900 50  0001 C CNN
+	1    6450 2900
 	1    0    0    -1
 $EndComp
@@
 F 0 "D4" V 1954 5679 50  0000 L CNN
 F 1 "D_TVS" V 2045 5679 50  0000 L CNN
-F 2 "Diode_THT:D_DO-15_P10.16mm_Horizontal" H 2000 5600 50  0001 C CNN
+F 2 "Diode_SMD:D_0201_0603Metric" H 2000 5600 50  0001 C CNN
 F 3 "~" H 2000 5600 50  0001 C CNN
 	1    2000 5600
@@
 L power:GND #PWR023
 U 1 1 5DCAAD30
-P 2500 5800
-F 0 "#PWR023" H 2500 5550 50  0001 C CNN
-F 1 "GND" H 2505 5627 50  0000 C CNN
-F 2 "" H 2500 5800 50  0001 C CNN
-F 3 "" H 2500 5800 50  0001 C CNN
-	1    2500 5800
+P 2500 6000
+F 0 "#PWR023" H 2500 5750 50  0001 C CNN
+F 1 "GND" H 2505 5827 50  0000 C CNN
+F 2 "" H 2500 6000 50  0001 C CNN
+F 3 "" H 2500 6000 50  0001 C CNN
+	1    2500 6000
 	1    0    0    -1
 $EndComp
@@
 L Device:C C13
 U 1 1 5DCAAD47
-P 3750 6850
-F 0 "C13" H 3635 6896 50  0000 R CNN
-F 1 "0.1uF-50V" H 3635 6805 50  0000 R CNN
-F 2 "Capacitor_SMD:C_0805_2012Metric" H 3788 6700 50  0001 C CNN
-F 3 "~" H 3750 6850 50  0001 C CNN
-	1    3750 6850
+P 3250 6700
+F 0 "C13" H 3135 6746 50  0000 R CNN
+F 1 "0.1uF-50V" H 3135 6655 50  0000 R CNN
+F 2 "Capacitor_SMD:C_0805_2012Metric" H 3288 6550 50  0001 C CNN
+F 3 "~" H 3250 6700 50  0001 C CNN
+	1    3250 6700
 	-1   0    0    -1
 $EndComp
@@
 L Device:C C15
 U 1 1 5E259978
-P 4400 6850
-F 0 "C15" H 4515 6896 50  0000 L CNN
-F 1 "0.1uF-50V" H 4515 6805 50  0000 L CNN
-F 2 "Capacitor_SMD:C_0805_2012Metric" H 4438 6700 50  0001 C CNN
-F 3 "~" H 4400 6850 50  0001 C CNN
-	1    4400 6850
+P 3250 7100
+F 0 "C15" H 3365 7146 50  0000 L CNN
+F 1 "0.1uF-50V" H 3365 7055 50  0000 L CNN
+F 2 "Capacitor_SMD:C_0805_2012Metric" H 3288 6950 50  0001 C CNN
+F 3 "~" H 3250 7100 50  0001 C CNN
+	1    3250 7100
 	1    0    0    -1
 $EndComp
@@
 L power:GND #PWR033
 U 1 1 5E25997E
-P 4100 7000
-F 0 "#PWR033" H 4100 6750 50  0001 C CNN
-F 1 "GND" H 4105 6827 50  0000 C CNN
-F 2 "" H 4100 7000 50  0001 C CNN
-F 3 "" H 4100 7000 50  0001 C CNN
-	1    4100 7000
+P 3000 6950
+F 0 "#PWR033" H 3000 6700 50  0001 C CNN
+F 1 "GND" H 3005 6777 50  0000 C CNN
+F 2 "" H 3000 6950 50  0001 C CNN
+F 3 "" H 3000 6950 50  0001 C CNN
+	1    3000 6950
 	1    0    0    -1
 $EndComp
@@
 L power:-12V #PWR035
 U 1 1 5E25998A
-P 4400 6650
-F 0 "#PWR035" H 4400 6750 50  0001 C CNN
-F 1 "-12V" H 4415 6823 50  0000 C CNN
-F 2 "" H 4400 6650 50  0001 C CNN
-F 3 "" H 4400 6650 50  0001 C CNN
-	1    4400 6650
-	1    0    0    -1
-$EndComp
-Wire Wire Line
-	3750 7000 4100 7000
+P 3250 7350
+F 0 "#PWR035" H 3250 7450 50  0001 C CNN
+F 1 "-12V" H 3265 7523 50  0000 C CNN
+F 2 "" H 3250 7350 50  0001 C CNN
+F 3 "" H 3250 7350 50  0001 C CNN
+	1    3250 7350
+	-1   0    0    1
+$EndComp
 Wire Wire Line
 	5700 4950 5700 4650
@@
 ARP
 Wire Wire Line
-	4400 6650 4400 6700
-Wire Wire Line
-	3750 6650 3750 6700
-Wire Wire Line
-	4100 7000 4400 7000
-Connection ~ 4100 7000
+	3250 6500 3250 6550
 Wire Wire Line
 	5700 3650 5700 4650
@@
 	5700 4650 6600 4650
 Wire Wire Line
-	3700 950  3700 1000
-Wire Wire Line
-	4400 950  4400 1000
-Wire Wire Line
-	4100 1300 4400 1300
-Connection ~ 4100 1300
+	3150 900  3150 950
 $Comp
 L Device:C C17
@@
 L power:GND #PWR043
 U 1 1 5E37BE4D
-P 6600 5150
-F 0 "#PWR043" H 6600 4900 50  0001 C CNN
-F 1 "GND" H 6605 4977 50  0000 C CNN
-F 2 "" H 6600 5150 50  0001 C CNN
-F 3 "" H 6600 5150 50  0001 C CNN
-	1    6600 5150
+P 6450 5300
+F 0 "#PWR043" H 6450 5050 50  0001 C CNN
+F 1 "GND" H 6455 5127 50  0000 C CNN
+F 2 "" H 6450 5300 50  0001 C CNN
+F 3 "" H 6450 5300 50  0001 C CNN
+	1    6450 5300
 	1    0    0    -1
 $EndComp
@@
 L power:+12V #PWR031
 U 1 1 5DCAAD37
-P 3750 6650
-F 0 "#PWR031" H 3750 6500 50  0001 C CNN
-F 1 "+12V" H 3765 6823 50  0000 C CNN
-F 2 "" H 3750 6650 50  0001 C CNN
-F 3 "" H 3750 6650 50  0001 C CNN
-	1    3750 6650
+P 3250 6500
+F 0 "#PWR031" H 3250 6350 50  0001 C CNN
+F 1 "+12V" H 3265 6673 50  0000 C CNN
+F 2 "" H 3250 6500 50  0001 C CNN
+F 3 "" H 3250 6500 50  0001 C CNN
+	1    3250 6500
 	1    0    0    -1
 $EndComp
@@
 Wire Notes Line
 	11000 4700 9250 4700
+Wire Wire Line
+	2500 3100 2500 3300
+Wire Wire Line
+	2500 5800 2500 6000
+Wire Wire Line
+	6600 2750 6450 2750
+Wire Wire Line
+	6450 2750 6450 2900
+Wire Wire Line
+	6600 5150 6450 5150
+Wire Wire Line
+	6450 5150 6450 5300
+Text Notes 750  3600 0    50   ~ 0
+JP3\nSelección de Carga de Entrada R3\n\n
+Text Notes 800  6400 0    50   ~ 0
+JP4\nSelección de Carga de Entrada R4\n\n
+Text Notes 5450 3600 2    50   ~ 0
+JP5\nSelección salida negada\n\n
+Text Notes 5450 6400 2    50   ~ 0
+JP6\nSelección salida negada\n\n
+Wire Wire Line
+	3250 6850 3250 6900
+Wire Wire Line
+	3250 6900 3000 6900
+Wire Wire Line
+	3000 6900 3000 6950
+Wire Wire Line
+	3250 6900 3250 6950
+Connection ~ 3250 6900
+Wire Wire Line
+	3250 7250 3250 7350
+Wire Wire Line
+	3150 1250 3150 1300
+Wire Wire Line
+	3150 1650 3150 1750
+Wire Wire Line
+	3150 1300 2800 1300
+Wire Wire Line
+	2800 1300 2800 1400
+Connection ~ 3150 1300
+Wire Wire Line
+	3150 1300 3150 1350
 $EndSCHEMATC

Commit message: mejorando BOM - work in progress
Parts:
- U11, U12: Número de Parte (Digi-Key) (none) -> 296-47682-1-ND
- U21, U22: Descripción (inglés) Dual 2.7-V High Slew Rate Rail-To-Rail Output Operational A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 -> General Purpose Amplifier 2 Circuit Rail-to-Rail 8-SOIC; Enlace https://www.digikey.com/product-detail/en/texas-instruments/TLV2772IDR/296-1902-1-ND/405014?utm_source=snapeda&utm_medium=aggregator&utm_campaign=symbol -> https://www.digikey.com/product-detail/en/texas-instruments/TLV2772IDR/296-1902-2-ND/374332; Número de Parte (Digi-Key) 296-1902-1-ND -> 296-1902-2-ND; Número de parte (Digi-Key) (none) -> 296-1902-2-ND
- U31: Descripción (inglés) (none) -> Dual-Bit Dual-Supply Bus Transceiver With Configurable Volt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; Enlace (none) -> https://www.digikey.com/product-detail/en/texas-instruments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; Fabricante (none) -> Texas Instruments; Número de Parte (Digi-Key) (none) -> 296-17014-1-ND; Número de parte (Digi-Key) (none) -> 296-17014-1-ND
Changed lines of the file:
@@
 F 6 "296-47682-1-ND" H 4100 2500 50  0001 L BNN "Número de parte (Digi-Key)"
 F 7 "https://www.digikey.com/product-detail/en/texas-instruments/LM361MX-NOPB/296-47682-1-ND/3526971" H 4100 2500 50  0001 L BNN "Enlace"
+F 8 "296-47682-1-ND" H 4100 2500 50  0001 C CNN "Número de Parte (Digi-Key)"
 	1    4100 2500
 	1    0    0    -1
@@
 F 3 "http://www.ti.com/lit/ds/symlink/tlv2772.pdf" H 7300 2250 50  0001 L BNN
 F 4 "Texas Instruments" H 7300 2250 50  0001 L BNN "Fabricante"
-F 5 "Dual 2.7-V High Slew Rate Rail-To-Rail Output Operational Amplifier 8-SOIC -40 to 125" H 7300 2250 50  0001 L BNN "Descripción (inglés)"
-F 6 "296-1902-1-ND" H 7300 2250 50  0001 L BNN "Número de Parte (Digi-Key)"
-F 7 "https://www.digikey.com/product-detail/en/texas-instruments/TLV2772IDR/296-1902-1-ND/405014?utm_source=snapeda&utm_medium=aggregator&utm_campaign=symbol" H 7300 2250 50  0001 L BNN "Enlace"
+F 5 "General Purpose Amplifier 2 Circuit Rail-to-Rail 8-SOIC" H 7300 2250 50  0001 L BNN "Descripción (inglés)"
+F 6 "296-1902-2-ND" H 7300 2250 50  0001 L BNN "Número de Parte (Digi-Key)"
+F 7 "https://www.digikey.com/product-detail/en/texas-instruments/TLV2772IDR/296-1902-2-ND/374332" H 7300 2250 50  0001 L BNN "Enlace"
+F 8 "296-1902-2-ND" H 7300 2250 50  0001 C CNN "Número de parte (Digi-Key)"
 	1    7300 2250
 	1    0    0    -1
@@
 F 2 "Package_SO:VSSOP-8_2.4x2.1mm_P0.5mm" H 9850 3000 50  0001 C CNN
 F 3 "http://www.ti.com/lit/ds/symlink/sn74lvc2t45.pdf" H 8900 3000 50  0001 C CNN
+F 4 "Dual-Bit Dual-Supply Bus Transceiver With Configurable Voltage" H 9800 3550 50  0001 C CNN "Descripción (inglés)"
+F 5 "https://www.digikey.com/product-detail/en/texas-instruments/SN74LVC2T45DCUR/296-17014-2-ND/657833" H 9800 3550 50  0001 C CNN "Enlace"
+F 6 "Texas Instruments" H 9800 3550 50  0001 C CNN "Fabricante"
+F 7 "296-17014-1-ND" H 9800 3550 50  0001 C CNN "Número de Parte (Digi-Key)"
+F 8 "296-17014-1-ND" H 9800 3550 50  0001 C CNN "Número de parte (Digi-Key)"
 	1    9800 3550
 	-1   0    0    -1
@@
 F 6 "296-47682-1-ND" H 4100 5200 50  0001 L BNN "Número de parte (Digi-Key)"
 F 7 "https://www.digikey.com/product-detail/en/texas-instruments/LM361MX-NOPB/296-47682-1-ND/3526971" H 4100 5200 50  0001 L BNN "Enlace"
+F 8 "296-47682-1-ND" H 4100 5200 50  0001 C CNN "Número de Parte (Digi-Key)"
 	1    4100 5200
 	1    0    0    -1
@@
 F 3 "http://www.ti.com/lit/ds/symlink/tlv2772.pdf" H 7300 4650 50  0001 L BNN
 F 4 "Texas Instruments" H 7300 4650 50  0001 L BNN "Fabricante"
-F 5 "Dual 2.7-V High Slew Rate Rail-To-Rail Output Operational Amplifier 8-SOIC -40 to 125" H 7300 4650 50  0001 L BNN "Descripción (inglés)"
-F 6 "296-1902-1-ND" H 7300 4650 50  0001 L BNN "Número de Parte (Digi-Key)"
-F 7 "https://www.digikey.com/product-detail/en/texas-instruments/TLV2772IDR/296-1902-1-ND/405014?utm_source=snapeda&utm_medium=aggregator&utm_campaign=symbol" H 7300 4650 50  0001 L BNN "Enlace"
+F 5 "General Purpose Amplifier 2 Circuit Rail-to-Rail 8-SOIC" H 7300 4650 50  0001 L BNN "Descripción (inglés)"
+F 6 "296-1902-2-ND" H 7300 4650 50  0001 L BNN "Número de Parte (Digi-Key)"
+F 7 "https://www.digikey.com/product-detail/en/texas-instruments/TLV2772IDR/296-1902-2-ND/374332" H 7300 4650 50  0001 L BNN "Enlace"
+F 8 "296-1902-2-ND" H 7300 4650 50  0001 C CNN "Número de parte (Digi-Key)"
 	1    7300 4650
 	1    0    0    -1
