File: adaptadora/prf_y_sec.sch (KiCad schematic (older format))
At the start: 39 parts

Commit message: correcciones implementadas
Parts:
- removed C? (x4): 0.1uF-50V, symbol Device:C
- removed C?: 1uF-16V, symbol Device:CP1
- removed J? (x4): Conn_Coaxial, symbol Connector:Conn_Coaxial
- removed JP? (x2): Jumper_3_Open, symbol Jumper:Jumper_3_Open
- removed R?: 100 - 1/8W - 5%, symbol Device:R
- removed RV?: R_POT, symbol Device:R_POT
- removed U? (x2): TLV2772IDR, SOIC127P600X175-8N, symbol TLV2772IDR:TLV2772IDR
- added C20: 1uF-16V, symbol Device:CP1
- added C23, C24, C27, C30: 0.1uF-50V, symbol Device:C
- added J20, J21, J22, J23: Conn_Coaxial, symbol Connector:Conn_Coaxial
- added JP10, JP9: Jumper_3_Open, symbol Jumper:Jumper_3_Open
- added R9: 100 - 1/8W - 5%, symbol Device:R
- added RV7: R_POT, symbol Device:R_POT
- added U2_3, U2_4: TLV2772IDR, SOIC127P600X175-8N, symbol TLV2772IDR:TLV2772IDR
- U1_1: renamed from U?; Campo4 Unavailable -> (none); Campo5 None -> (none); Campo6 LM361MX/NOPB -> (none); Campo7 High Speed Differential Comparator 14-SOIC 0 to 70 -> (none); Campo8 Texas Instruments -> (none); Descripción (inglés) (none) -> High Speed Differential Comparator 14-SOIC 0 to 70; Enlace (none) -> https://www.digikey.com/product-detail/en/texas-instruments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; Fabricante (none) -> Texas Instruments; Número de parte (Digi-Key) (none) -> 296-47682-1-ND
- gave numbers to parts that had none: 22
Connections:
- net +12V: now also C24.1
- net +5V: now also C23.2, C30.2, U2_3.8 (VDD), U2_4.8 (VDD)
- net -12V: now also C27.1
- net GND: now also C20.2, C23.1, C24.2, C27.2, C30.1, J20.2 (Ext), J21.2 (Ext), J22.2 (Ext), J23.2 (Ext), RV7.3, U2_3.4 (GND), U2_4.4 (GND)
- net PRF: now also JP9.2 (C), U2_3.3 (1IN+), U2_3.5 (2IN+)
- net VIDEO_COMP: now also JP10.2 (C), U2_4.3 (1IN+), U2_4.5 (2IN+)
- net at RV9.2, U1_1.4 (-IN): now also C20.1
- net at J18.1 (In), JP7.1 (A): now also RV7.1
- net at D5.1 (A1): now also R9.2, RV7.2
- net at U1_1.11 (OUT+): now also JP9.1 (A)
- net at U1_1.3 (+IN): now also R9.1
- net at U1_1.9 (OUT-): now also JP9.3 (B)
- net at U1_1.11 (OUT+): now also JP10.1 (A)
- net at U1_1.9 (OUT-): now also JP10.3 (B)
- net VIDEO_COMP_3P3 renamed V_COMP_3P3
- new net: J22.1 (In), U2_3.1 (1OUT), U2_3.2 (1IN-)
- new net: J20.1 (In), U2_3.6 (2IN-), U2_3.7 (2OUT)
- new net: J23.1 (In), U2_4.1 (1OUT), U2_4.2 (1IN-)
- new net: J21.1 (In), U2_4.6 (2IN-), U2_4.7 (2OUT)
Other:
- note added: "U1_X: Comparadores\nTensión de señal de entrada máxima 12 V\nTensión de señal de salida 5V"
- note added: "U2_X: Amplificadores operacionales\nSalidas duplicadas para otros equipos\nTensión de salida: 5V"
- note added: "U3_X: Convertidor de Niveles Lógicos\nTensión de señal de entrada 5 V\nTensión de señal de salida 3.3V"

Commit message: se agregan huellas, en progreso
Parts:
- J18, J19, J20, J21, J22, J23: footprint (none) -> Connector_Coaxial:SMA_Amphenol_901-144_Vertical
- renumbered U1_1 to U1_2
Changed lines of the file:
@@
 F 0 "J18" H 628 2188 50  0000 C CNN
 F 1 "Conn_Coaxial" H 628 2097 50  0000 C CNN
-F 2 "" H 700 1950 50  0001 C CNN
+F 2 "Connector_Coaxial:SMA_Amphenol_901-144_Vertical" H 700 1950 50  0001 C CNN
 F 3 " ~" H 700 1950 50  0001 C CNN
 	1    700  1950
@@
 F 0 "J19" H 628 4888 50  0000 C CNN
 F 1 "Conn_Coaxial" H 628 4797 50  0000 C CNN
-F 2 "" H 700 4650 50  0001 C CNN
+F 2 "Connector_Coaxial:SMA_Amphenol_901-144_Vertical" H 700 4650 50  0001 C CNN
 F 3 " ~" H 700 4650 50  0001 C CNN
 	1    700  4650
@@
 	950  5800 1850 5800
 $Comp
-L sincronismo-rescue:LM361MX_NOPB-LM361MX_NOPB U1_1
+L sincronismo-rescue:LM361MX_NOPB-LM361MX_NOPB U1_2
 U 1 1 5DC9BD27
 P 4100 5200
-F 0 "U1_1" H 4100 5870 50  0000 C CNN
+F 0 "U1_2" H 4100 5870 50  0000 C CNN
 F 1 "LM361MX_NOPB" H 4100 5779 50  0000 C CNN
 F 2 "SOIC127P600X175-14N" H 4100 5200 50  0001 L BNN
@@
 F 0 "J23" H 8800 4325 50  0000 L CNN
 F 1 "Conn_Coaxial" H 8800 4234 50  0000 L CNN
-F 2 "" H 8700 4350 50  0001 C CNN
+F 2 "Connector_Coaxial:SMA_Amphenol_901-144_Vertical" H 8700 4350 50  0001 C CNN
 F 3 " ~" H 8700 4350 50  0001 C CNN
 	1    8700 4350
@@
 F 0 "J21" H 8100 4550 50  0000 L CNN
 F 1 "Conn_Coaxial" H 7850 4450 50  0000 L CNN
-F 2 "" H 8450 4650 50  0001 C CNN
+F 2 "Connector_Coaxial:SMA_Amphenol_901-144_Vertical" H 8450 4650 50  0001 C CNN
 F 3 " ~" H 8450 4650 50  0001 C CNN
 	1    8450 4650
@@
 F 0 "J22" H 8800 1925 50  0000 L CNN
 F 1 "Conn_Coaxial" H 8800 1834 50  0000 L CNN
-F 2 "" H 8700 1950 50  0001 C CNN
+F 2 "Connector_Coaxial:SMA_Amphenol_901-144_Vertical" H 8700 1950 50  0001 C CNN
 F 3 " ~" H 8700 1950 50  0001 C CNN
 	1    8700 1950
@@
 F 0 "J20" H 8100 2150 50  0000 L CNN
 F 1 "Conn_Coaxial" H 7850 2050 50  0000 L CNN
-F 2 "" H 8450 2250 50  0001 C CNN
+F 2 "Connector_Coaxial:SMA_Amphenol_901-144_Vertical" H 8450 2250 50  0001 C CNN
 F 3 " ~" H 8450 2250 50  0001 C CNN
 	1    8450 2250

Commit message: pcb work in progress
Parts:
- C20, C21: footprint (none) -> Resistor_SMD:R_1206_3216Metric
- C22, C23, C24, C25, C26, C27, C28, C29, C30, C31: footprint (none) -> Capacitor_SMD:C_0805_2012Metric
- D5, D6: footprint (none) -> Diode_THT:D_DO-15_P10.16mm_Horizontal
- JP10, JP7, JP8, JP9: footprint (none) -> Jumper:SolderJumper-3_P1.3mm_Open_Pad1.0x1.5mm_NumberLabels
- R10, R9: footprint (none) -> Resistor_SMD:R_0805_2012Metric
- R7, R8: footprint (none) -> Resistor_THT:R_Axial_DIN0414_L11.9mm_D4.5mm_P15.24mm_Horizontal
- RV10, RV7, RV8, RV9: footprint (none) -> Potentiometer_THT:Potentiometer_Bourns_3296W_Vertical
- TP3, TP4: footprint (none) -> TestPoint:TestPoint_THTPad_1.5x1.5mm_Drill0.7mm
- U13: renamed from U1_1; footprint SOIC127P600X175-14N -> Package_DIP:DIP-14_W7.62mm
- U14: renamed from U1_2; footprint SOIC127P600X175-14N -> Package_DIP:DIP-14_W7.62mm
- U23: renamed from U2_3; footprint SOIC127P600X175-8N -> Package_SO:SOIC-8_7.5x5.85mm_P1.27mm
- U24: renamed from U2_4; footprint SOIC127P600X175-8N -> Package_SO:SOIC-8_7.5x5.85mm_P1.27mm
- renumbered U3_2 to U32
Changed lines of the file:
@@
 F 0 "RV7" H 1781 2246 50  0000 R CNN
 F 1 "R_POT" H 1781 2155 50  0000 R CNN
-F 2 "" H 1850 2200 50  0001 C CNN
+F 2 "Potentiometer_THT:Potentiometer_Bourns_3296W_Vertical" H 1850 2200 50  0001 C CNN
 F 3 "~" H 1850 2200 50  0001 C CNN
 	1    1850 2200
@@
 F 0 "D5" V 1954 2979 50  0000 L CNN
 F 1 "D_TVS" V 2045 2979 50  0000 L CNN
-F 2 "" H 2000 2900 50  0001 C CNN
+F 2 "Diode_THT:D_DO-15_P10.16mm_Horizontal" H 2000 2900 50  0001 C CNN
 F 3 "~" H 2000 2900 50  0001 C CNN
 	1    2000 2900
@@
 F 0 "C20" H 2765 2946 50  0000 L CNN
 F 1 "1uF-16V" H 2765 2855 50  0000 L CNN
-F 2 "" H 2650 2900 50  0001 C CNN
+F 2 "Resistor_SMD:R_1206_3216Metric" H 2650 2900 50  0001 C CNN
 F 3 "~" H 2650 2900 50  0001 C CNN
 	1    2650 2900
@@
 F 0 "R9" V 2093 2200 50  0000 C CNN
 F 1 "100 - 1/8W - 5%" V 2184 2200 50  0000 C CNN
-F 2 "" V 2230 2200 50  0001 C CNN
+F 2 "Resistor_SMD:R_0805_2012Metric" V 2230 2200 50  0001 C CNN
 F 3 "~" H 2300 2200 50  0001 C CNN
 	1    2300 2200
@@
 F 0 "R7" H 1020 2896 50  0000 L CNN
 F 1 "50 - 1/2W - 5%" H 1020 2805 50  0000 L CNN
-F 2 "" V 880 2850 50  0001 C CNN
+F 2 "Resistor_THT:R_Axial_DIN0414_L11.9mm_D4.5mm_P15.24mm_Horizontal" V 880 2850 50  0001 C CNN
 F 3 "~" H 950 2850 50  0001 C CNN
 	1    950  2850
@@
 F 0 "JP7" V 1054 2487 50  0000 L CNN
 F 1 "Jumper_3_Open" V 1145 2487 50  0000 L CNN
-F 2 "" H 1100 2400 50  0001 C CNN
+F 2 "Jumper:SolderJumper-3_P1.3mm_Open_Pad1.0x1.5mm_NumberLabels" H 1100 2400 50  0001 C CNN
 F 3 "~" H 1100 2400 50  0001 C CNN
 	1    1100 2400
@@
 F 0 "C22" H 3400 3200 50  0000 R CNN
 F 1 "0.1uF-50V" H 3550 3300 50  0000 R CNN
-F 2 "" H 3388 2800 50  0001 C CNN
+F 2 "Capacitor_SMD:C_0805_2012Metric" H 3388 2800 50  0001 C CNN
 F 3 "~" H 3350 2950 50  0001 C CNN
 	1    3350 2950
@@
 	950  3100 1850 3100
 $Comp
-L sincronismo-rescue:LM361MX_NOPB-LM361MX_NOPB U1_1
+L sincronismo-rescue:LM361MX_NOPB-LM361MX_NOPB U13
 U 1 1 5DC9BCFB
 P 4100 2500
-F 0 "U1_1" H 4100 3170 50  0000 C CNN
+F 0 "U13" H 4100 3170 50  0000 C CNN
 F 1 "LM361MX_NOPB" H 4100 3079 50  0000 C CNN
-F 2 "SOIC127P600X175-14N" H 4100 2500 50  0001 L BNN
+F 2 "Package_DIP:DIP-14_W7.62mm" H 4100 2500 50  0001 L BNN
 F 3 "SOIC-14 Texas Instruments" H 4100 2500 50  0001 L BNN
 F 4 "Texas Instruments" H 4100 2500 50  0001 L BNN "Fabricante"
@@
 F 0 "JP9" V 5354 2337 50  0000 L CNN
 F 1 "Jumper_3_Open" V 5445 2337 50  0000 L CNN
-F 2 "" H 5400 2250 50  0001 C CNN
+F 2 "Jumper:SolderJumper-3_P1.3mm_Open_Pad1.0x1.5mm_NumberLabels" H 5400 2250 50  0001 C CNN
 F 3 "~" H 5400 2250 50  0001 C CNN
 	1    5400 2250
@@
 F 0 "TP3" H 5758 1368 50  0000 L CNN
 F 1 "TestPoint" H 5758 1277 50  0000 L CNN
-F 2 "" H 5900 1250 50  0001 C CNN
+F 2 "TestPoint:TestPoint_THTPad_1.5x1.5mm_Drill0.7mm" H 5900 1250 50  0001 C CNN
 F 3 "~" H 5900 1250 50  0001 C CNN
 	1    5700 1250
@@
 F 0 "C24" H 3900 1050 50  0000 R CNN
 F 1 "0.1uF-50V" H 3700 900 50  0000 L BNN
-F 2 "" H 3738 1000 50  0001 C CNN
+F 2 "Capacitor_SMD:C_0805_2012Metric" H 3738 1000 50  0001 C CNN
 F 3 "~" H 3700 1150 50  0001 C CNN
 	1    3700 1150
@@
 F 0 "C26" H 4150 1250 50  0000 L CNN
 F 1 "0.1uF-50V" H 3900 1150 50  0000 L CNN
-F 2 "" H 4438 1000 50  0001 C CNN
+F 2 "Capacitor_SMD:C_0805_2012Metric" H 4438 1000 50  0001 C CNN
 F 3 "~" H 4400 1150 50  0001 C CNN
 	1    4400 1150
@@
 $EndComp
 $Comp
-L TLV2772IDR:TLV2772IDR U2_3
+L TLV2772IDR:TLV2772IDR U23
 U 1 1 5DCAAD22
 P 7300 2250
-F 0 "U2_3" H 7300 2820 50  0000 C CNN
+F 0 "U23" H 7300 2820 50  0000 C CNN
 F 1 "TLV2772IDR" H 7300 2729 50  0000 C CNN
-F 2 "SOIC127P600X175-8N" H 7300 2250 50  0001 L BNN
+F 2 "Package_SO:SOIC-8_7.5x5.85mm_P1.27mm" H 7300 2250 50  0001 L BNN
 F 3 "296-1902-1-ND" H 7300 2250 50  0001 L BNN
 F 4 "Texas Instruments" H 7300 2250 50  0001 L BNN "Campo4"
@@
 F 0 "C31" V 9950 2650 50  0000 C CNN
 F 1 "0.1uF-50V" V 10300 2600 50  0000 C CNN
-F 2 "" H 10188 2500 50  0001 C CNN
+F 2 "Capacitor_SMD:C_0805_2012Metric" H 10188 2500 50  0001 C CNN
 F 3 "~" H 10150 2650 50  0001 C CNN
 	1    10150 2650
@@
 $EndComp
 $Comp
-L Logic_LevelTranslator:SN74LVC2T45DCUR U3_2
+L Logic_LevelTranslator:SN74LVC2T45DCUR U32
 U 1 1 5DA3673D
 P 9800 3550
-F 0 "U3_2" H 9800 2961 50  0000 C CNN
+F 0 "U32" H 9800 2961 50  0000 C CNN
 F 1 "SN74LVC2T45DCUR" H 9800 2870 50  0000 C CNN
 F 2 "Package_SO:VSSOP-8_2.4x2.1mm_P0.5mm" H 9850 3000 50  0001 C CNN
@@
 F 0 "C28" H 6200 1750 50  0000 L CNN
 F 1 "0.1uF-50V" H 5950 1650 50  0000 L CNN
-F 2 "" H 6488 1700 50  0001 C CNN
+F 2 "Capacitor_SMD:C_0805_2012Metric" H 6488 1700 50  0001 C CNN
 F 3 "~" H 6450 1850 50  0001 C CNN
 	1    6450 1850
@@
 F 0 "RV8" H 1781 4946 50  0000 R CNN
 F 1 "R_POT" H 1781 4855 50  0000 R CNN
-F 2 "" H 1850 4900 50  0001 C CNN
+F 2 "Potentiometer_THT:Potentiometer_Bourns_3296W_Vertical" H 1850 4900 50  0001 C CNN
 F 3 "~" H 1850 4900 50  0001 C CNN
 	1    1850 4900
@@
 F 0 "D6" V 1954 5679 50  0000 L CNN
 F 1 "D_TVS" V 2045 5679 50  0000 L CNN
-F 2 "" H 2000 5600 50  0001 C CNN
+F 2 "Diode_THT:D_DO-15_P10.16mm_Horizontal" H 2000 5600 50  0001 C CNN
 F 3 "~" H 2000 5600 50  0001 C CNN
 	1    2000 5600
@@
 F 0 "RV10" H 2431 5396 50  0000 R CNN
 F 1 "R_POT" H 2431 5305 50  0000 R CNN
-F 2 "" H 2500 5350 50  0001 C CNN
+F 2 "Potentiometer_THT:Potentiometer_Bourns_3296W_Vertical" H 2500 5350 50  0001 C CNN
 F 3 "~" H 2500 5350 50  0001 C CNN
 	1    2500 5350
@@
 F 0 "C21" H 2765 5646 50  0000 L CNN
 F 1 "1uF-16V" H 2765 5555 50  0000 L CNN
-F 2 "" H 2650 5600 50  0001 C CNN
+F 2 "Resistor_SMD:R_1206_3216Metric" H 2650 5600 50  0001 C CNN
 F 3 "~" H 2650 5600 50  0001 C CNN
 	1    2650 5600
@@
 F 0 "R10" V 2093 4900 50  0000 C CNN
 F 1 "100 - 1/8W - 5%" V 2184 4900 50  0000 C CNN
-F 2 "" V 2230 4900 50  0001 C CNN
+F 2 "Resistor_SMD:R_0805_2012Metric" V 2230 4900 50  0001 C CNN
 F 3 "~" H 2300 4900 50  0001 C CNN
 	1    2300 4900
@@
 F 0 "R8" H 1020 5596 50  0000 L CNN
 F 1 "50 - 1/2W - 5%" H 1020 5505 50  0000 L CNN
-F 2 "" V 880 5550 50  0001 C CNN
+F 2 "Resistor_THT:R_Axial_DIN0414_L11.9mm_D4.5mm_P15.24mm_Horizontal" V 880 5550 50  0001 C CNN
 F 3 "~" H 950 5550 50  0001 C CNN
 	1    950  5550
@@
 F 0 "JP8" V 1054 5187 50  0000 L CNN
 F 1 "Jumper_3_Open" V 1145 5187 50  0000 L CNN
-F 2 "" H 1100 5100 50  0001 C CNN
+F 2 "Jumper:SolderJumper-3_P1.3mm_Open_Pad1.0x1.5mm_NumberLabels" H 1100 5100 50  0001 C CNN
 F 3 "~" H 1100 5100 50  0001 C CNN
 	1    1100 5100
@@
 F 0 "C23" H 3400 5900 50  0000 R CNN
 F 1 "0.1uF-50V" H 3550 6000 50  0000 R CNN
-F 2 "" H 3388 5500 50  0001 C CNN
+F 2 "Capacitor_SMD:C_0805_2012Metric" H 3388 5500 50  0001 C CNN
 F 3 "~" H 3350 5650 50  0001 C CNN
 	1    3350 5650
@@
 	950  5800 1850 5800
 $Comp
-L sincronismo-rescue:LM361MX_NOPB-LM361MX_NOPB U1_2
+L sincronismo-rescue:LM361MX_NOPB-LM361MX_NOPB U14
 U 1 1 5DC9BD27
 P 4100 5200
-F 0 "U1_2" H 4100 5870 50  0000 C CNN
+F 0 "U14" H 4100 5870 50  0000 C CNN
 F 1 "LM361MX_NOPB" H 4100 5779 50  0000 C CNN
-F 2 "SOIC127P600X175-14N" H 4100 5200 50  0001 L BNN
+F 2 "Package_DIP:DIP-14_W7.62mm" H 4100 5200 50  0001 L BNN
 F 3 "SOIC-14 Texas Instruments" H 4100 5200 50  0001 L BNN
 F 4 "Texas Instruments" H 4100 5200 50  0001 L BNN "Fabricante"
@@
 F 0 "JP10" V 5354 5037 50  0000 L CNN
 F 1 "Jumper_3_Open" V 5445 5037 50  0000 L CNN
-F 2 "" H 5400 4950 50  0001 C CNN
+F 2 "Jumper:SolderJumper-3_P1.3mm_Open_Pad1.0x1.5mm_NumberLabels" H 5400 4950 50  0001 C CNN
 F 3 "~" H 5400 4950 50  0001 C CNN
 	1    5400 4950
@@
 F 0 "TP4" H 5642 5926 50  0000 R CNN
 F 1 "TestPoint" H 5642 6017 50  0000 R CNN
-F 2 "" H 5900 5900 50  0001 C CNN
+F 2 "TestPoint:TestPoint_THTPad_1.5x1.5mm_Drill0.7mm" H 5900 5900 50  0001 C CNN
 F 3 "~" H 5900 5900 50  0001 C CNN
 	1    5700 5900
@@
 F 0 "C25" H 3635 6896 50  0000 R CNN
 F 1 "0.1uF-50V" H 3635 6805 50  0000 R CNN
-F 2 "" H 3788 6700 50  0001 C CNN
+F 2 "Capacitor_SMD:C_0805_2012Metric" H 3788 6700 50  0001 C CNN
 F 3 "~" H 3750 6850 50  0001 C CNN
 	1    3750 6850
@@
 F 0 "C27" H 4515 6896 50  0000 L CNN
 F 1 "0.1uF-50V" H 4515 6805 50  0000 L CNN
-F 2 "" H 4438 6700 50  0001 C CNN
+F 2 "Capacitor_SMD:C_0805_2012Metric" H 4438 6700 50  0001 C CNN
 F 3 "~" H 4400 6850 50  0001 C CNN
 	1    4400 6850
@@
 $EndComp
 $Comp
-L TLV2772IDR:TLV2772IDR U2_4
+L TLV2772IDR:TLV2772IDR U24
 U 1 1 5DCAAD4C
 P 7300 4650
-F 0 "U2_4" H 7300 5220 50  0000 C CNN
+F 0 "U24" H 7300 5220 50  0000 C CNN
 F 1 "TLV2772IDR" H 7300 5129 50  0000 C CNN
-F 2 "SOIC127P600X175-8N" H 7300 4650 50  0001 L BNN
+F 2 "Package_SO:SOIC-8_7.5x5.85mm_P1.27mm" H 7300 4650 50  0001 L BNN
 F 3 "296-1902-1-ND" H 7300 4650 50  0001 L BNN
 F 4 "Texas Instruments" H 7300 4650 50  0001 L BNN "Campo4"
@@
 F 0 "C29" H 6200 4250 50  0000 L CNN
 F 1 "0.1uF-50V" H 6000 4150 50  0000 L CNN
-F 2 "" H 6488 4100 50  0001 C CNN
+F 2 "Capacitor_SMD:C_0805_2012Metric" H 6488 4100 50  0001 C CNN
 F 3 "~" H 6450 4250 50  0001 C CNN
 	1    6450 4250
@@
 F 0 "C30" V 9250 2650 50  0000 C CNN
 F 1 "0.1uF-50V" V 9600 2700 50  0000 C CNN
-F 2 "" H 9488 2500 50  0001 C CNN
+F 2 "Capacitor_SMD:C_0805_2012Metric" H 9488 2500 50  0001 C CNN
 F 3 "~" H 9450 2650 50  0001 C CNN
 	1    9450 2650
@@
 F 0 "RV9" H 2431 2696 50  0000 R CNN
 F 1 "R_POT" H 2431 2605 50  0000 R CNN
-F 2 "" H 2500 2650 50  0001 C CNN
+F 2 "Potentiometer_THT:Potentiometer_Bourns_3296W_Vertical" H 2500 2650 50  0001 C CNN
 F 3 "~" H 2500 2650 50  0001 C CNN
 	1    2500 2650

Commit message: Componentes acomodados en PCB
Parts:
- U13, U14: footprint Package_DIP:DIP-14_W7.62mm -> Package_SO:SOIC-14_3.9x8.7mm_P1.27mm
- U23, U24: footprint Package_SO:SOIC-8_7.5x5.85mm_P1.27mm -> Package_SO:SOIC-8_3.9x4.9mm_P1.27mm
Changed lines of the file:
@@
 F 0 "U13" H 4100 3170 50  0000 C CNN
 F 1 "LM361MX_NOPB" H 4100 3079 50  0000 C CNN
-F 2 "Package_DIP:DIP-14_W7.62mm" H 4100 2500 50  0001 L BNN
+F 2 "Package_SO:SOIC-14_3.9x8.7mm_P1.27mm" H 4100 2500 50  0001 L BNN
 F 3 "SOIC-14 Texas Instruments" H 4100 2500 50  0001 L BNN
 F 4 "Texas Instruments" H 4100 2500 50  0001 L BNN "Fabricante"
@@
 F 0 "U23" H 7300 2820 50  0000 C CNN
 F 1 "TLV2772IDR" H 7300 2729 50  0000 C CNN
-F 2 "Package_SO:SOIC-8_7.5x5.85mm_P1.27mm" H 7300 2250 50  0001 L BNN
+F 2 "Package_SO:SOIC-8_3.9x4.9mm_P1.27mm" H 7300 2250 50  0001 L BNN
 F 3 "296-1902-1-ND" H 7300 2250 50  0001 L BNN
 F 4 "Texas Instruments" H 7300 2250 50  0001 L BNN "Campo4"
@@
 F 0 "U14" H 4100 5870 50  0000 C CNN
 F 1 "LM361MX_NOPB" H 4100 5779 50  0000 C CNN
-F 2 "Package_DIP:DIP-14_W7.62mm" H 4100 5200 50  0001 L BNN
+F 2 "Package_SO:SOIC-14_3.9x8.7mm_P1.27mm" H 4100 5200 50  0001 L BNN
 F 3 "SOIC-14 Texas Instruments" H 4100 5200 50  0001 L BNN
 F 4 "Texas Instruments" H 4100 5200 50  0001 L BNN "Fabricante"
@@
 F 0 "U24" H 7300 5220 50  0000 C CNN
 F 1 "TLV2772IDR" H 7300 5129 50  0000 C CNN
-F 2 "Package_SO:SOIC-8_7.5x5.85mm_P1.27mm" H 7300 4650 50  0001 L BNN
+F 2 "Package_SO:SOIC-8_3.9x4.9mm_P1.27mm" H 7300 4650 50  0001 L BNN
 F 3 "296-1902-1-ND" H 7300 4650 50  0001 L BNN
 F 4 "Texas Instruments" H 7300 4650 50  0001 L BNN "Campo4"
