File: adaptadora/prf_y_sec.sch (KiCad schematic (older format))
At the start: 39 parts, among them J18 Conn_Coaxial, J19 Conn_Coaxial, J20 Conn_Coaxial, J21 Conn_Coaxial, J22 Conn_Coaxial, J23 Conn_Coaxial, U13 LM361MX_NOPB, U14 LM361MX_NOPB, U23 TLV2772IDR, U24 TLV2772IDR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

Commit message: correcciones y archivos agregados
Parts:
- D5, D6: footprint Diode_THT:D_DO-15_P10.16mm_Horizontal -> Diode_SMD:D_0201_0603Metric
Connections:
- net -12V: now also C26.2, C27.2; no longer C26.1, C27.1
- net GND: now also C26.1, C27.1; no longer C26.2, C27.2
Other:
- note added: "JP10\nSelección de salida negada\n\n"
- note added: "JP7\nSelección de Carga de Entrada R7\n\n"
- note added: "JP8\nSelección de Carga de Entrada R8\n\n"
- note added: "JP9\nSelección salida negada\n\n"
- moved on the sheet: C24, C25, C26, C27
Changed lines of the file:
@@
 F 0 "D5" V 1954 2979 50  0000 L CNN
 F 1 "D_TVS" V 2045 2979 50  0000 L CNN
-F 2 "Diode_THT:D_DO-15_P10.16mm_Horizontal" H 2000 2900 50  0001 C CNN
+F 2 "Diode_SMD:D_0201_0603Metric" H 2000 2900 50  0001 C CNN
 F 3 "~" H 2000 2900 50  0001 C CNN
 	1    2000 2900
@@
 L power:GND #PWR051
 U 1 1 5DA58988
-P 2500 3100
-F 0 "#PWR051" H 2500 2850 50  0001 C CNN
-F 1 "GND" H 2505 2927 50  0000 C CNN
-F 2 "" H 2500 3100 50  0001 C CNN
-F 3 "" H 2500 3100 50  0001 C CNN
-	1    2500 3100
+P 2500 3350
+F 0 "#PWR051" H 2500 3100 50  0001 C CNN
+F 1 "GND" H 2505 3177 50  0000 C CNN
+F 2 "" H 2500 3350 50  0001 C CNN
+F 3 "" H 2500 3350 50  0001 C CNN
+	1    2500 3350
 	1    0    0    -1
 $EndComp
@@
 L Device:C C24
 U 1 1 5DCAAD13
-P 3700 1150
-F 0 "C24" H 3900 1050 50  0000 R CNN
-F 1 "0.1uF-50V" H 3700 900 50  0000 L BNN
-F 2 "Capacitor_SMD:C_0805_2012Metric" H 3738 1000 50  0001 C CNN
-F 3 "~" H 3700 1150 50  0001 C CNN
-	1    3700 1150
+P 3100 1000
+F 0 "C24" H 2900 1050 50  0000 R CNN
+F 1 "0.1uF-50V" H 2550 900 50  0000 L BNN
+F 2 "Capacitor_SMD:C_0805_2012Metric" H 3138 850 50  0001 C CNN
+F 3 "~" H 3100 1000 50  0001 C CNN
+	1    3100 1000
 	-1   0    0    -1
 $EndComp
@@
 L Device:C C26
 U 1 1 5DC9BD0B
-P 4400 1150
-F 0 "C26" H 4150 1250 50  0000 L CNN
-F 1 "0.1uF-50V" H 3900 1150 50  0000 L CNN
-F 2 "Capacitor_SMD:C_0805_2012Metric" H 4438 1000 50  0001 C CNN
-F 3 "~" H 4400 1150 50  0001 C CNN
-	1    4400 1150
+P 3100 1400
+F 0 "C26" H 3300 1500 50  0000 L CNN
+F 1 "0.1uF-50V" H 3200 1350 50  0000 L CNN
+F 2 "Capacitor_SMD:C_0805_2012Metric" H 3138 1250 50  0001 C CNN
+F 3 "~" H 3100 1400 50  0001 C CNN
+	1    3100 1400
 	1    0    0    -1
 $EndComp
@@
 L power:GND #PWR062
 U 1 1 5DCAAD14
-P 4100 1300
-F 0 "#PWR062" H 4100 1050 50  0001 C CNN
-F 1 "GND" H 4105 1127 50  0000 C CNN
-F 2 "" H 4100 1300 50  0001 C CNN
-F 3 "" H 4100 1300 50  0001 C CNN
-	1    4100 1300
+P 2750 1300
+F 0 "#PWR062" H 2750 1050 50  0001 C CNN
+F 1 "GND" H 2750 1100 50  0000 C CNN
+F 2 "" H 2750 1300 50  0001 C CNN
+F 3 "" H 2750 1300 50  0001 C CNN
+	1    2750 1300
 	1    0    0    -1
 $EndComp
@@
 L power:+12V #PWR060
 U 1 1 5DB62F12
-P 3700 950
-F 0 "#PWR060" H 3700 800 50  0001 C CNN
-F 1 "+12V" H 3715 1123 50  0000 C CNN
-F 2 "" H 3700 950 50  0001 C CNN
-F 3 "" H 3700 950 50  0001 C CNN
-	1    3700 950
-	1    0    0    -1
-$EndComp
-$Comp
-L power:-12V #PWR064
-U 1 1 5DB63B14
-P 4400 950
-F 0 "#PWR064" H 4400 1050 50  0001 C CNN
-F 1 "-12V" H 4415 1123 50  0000 C CNN
-F 2 "" H 4400 950 50  0001 C CNN
-F 3 "" H 4400 950 50  0001 C CNN
-	1    4400 950
-	1    0    0    -1
-$EndComp
-Wire Wire Line
-	3700 1300 4100 1300
+P 3100 800
+F 0 "#PWR060" H 3100 650 50  0001 C CNN
+F 1 "+12V" H 3115 973 50  0000 C CNN
+F 2 "" H 3100 800 50  0001 C CNN
+F 3 "" H 3100 800 50  0001 C CNN
+	1    3100 800
+	1    0    0    -1
+$EndComp
 $Comp
 L power:+5V #PWR070
@@
 L power:GND #PWR071
 U 1 1 5DC9BD17
-P 6600 2750
-F 0 "#PWR071" H 6600 2500 50  0001 C CNN
-F 1 "GND" H 6605 2577 50  0000 C CNN
-F 2 "" H 6600 2750 50  0001 C CNN
-F 3 "" H 6600 2750 50  0001 C CNN
-	1    6600 2750
+P 6450 2950
+F 0 "#PWR071" H 6450 2700 50  0001 C CNN
+F 1 "GND" H 6455 2777 50  0000 C CNN
+F 2 "" H 6450 2950 50  0001 C CNN
+F 3 "" H 6450 2950 50  0001 C CNN
+	1    6450 2950
 	1    0    0    -1
 $EndComp
@@
 F 0 "D6" V 1954 5679 50  0000 L CNN
 F 1 "D_TVS" V 2045 5679 50  0000 L CNN
-F 2 "Diode_THT:D_DO-15_P10.16mm_Horizontal" H 2000 5600 50  0001 C CNN
+F 2 "Diode_SMD:D_0201_0603Metric" H 2000 5600 50  0001 C CNN
 F 3 "~" H 2000 5600 50  0001 C CNN
 	1    2000 5600
@@
 L Device:C C25
 U 1 1 5E259972
-P 3750 6850
-F 0 "C25" H 3635 6896 50  0000 R CNN
-F 1 "0.1uF-50V" H 3635 6805 50  0000 R CNN
-F 2 "Capacitor_SMD:C_0805_2012Metric" H 3788 6700 50  0001 C CNN
-F 3 "~" H 3750 6850 50  0001 C CNN
-	1    3750 6850
+P 2900 6550
+F 0 "C25" H 2785 6596 50  0000 R CNN
+F 1 "0.1uF-50V" H 2785 6505 50  0000 R CNN
+F 2 "Capacitor_SMD:C_0805_2012Metric" H 2938 6400 50  0001 C CNN
+F 3 "~" H 2900 6550 50  0001 C CNN
+	1    2900 6550
 	-1   0    0    -1
 $EndComp
@@
 L Device:C C27
 U 1 1 5DCAAD48
-P 4400 6850
-F 0 "C27" H 4515 6896 50  0000 L CNN
-F 1 "0.1uF-50V" H 4515 6805 50  0000 L CNN
-F 2 "Capacitor_SMD:C_0805_2012Metric" H 4438 6700 50  0001 C CNN
-F 3 "~" H 4400 6850 50  0001 C CNN
-	1    4400 6850
+P 2900 6950
+F 0 "C27" H 3015 6996 50  0000 L CNN
+F 1 "0.1uF-50V" H 3015 6905 50  0000 L CNN
+F 2 "Capacitor_SMD:C_0805_2012Metric" H 2938 6800 50  0001 C CNN
+F 3 "~" H 2900 6950 50  0001 C CNN
+	1    2900 6950
 	1    0    0    -1
 $EndComp
@@
 L power:GND #PWR063
 U 1 1 5DCAAD49
-P 4100 7000
-F 0 "#PWR063" H 4100 6750 50  0001 C CNN
-F 1 "GND" H 4105 6827 50  0000 C CNN
-F 2 "" H 4100 7000 50  0001 C CNN
-F 3 "" H 4100 7000 50  0001 C CNN
-	1    4100 7000
+P 2600 6850
+F 0 "#PWR063" H 2600 6600 50  0001 C CNN
+F 1 "GND" H 2605 6677 50  0000 C CNN
+F 2 "" H 2600 6850 50  0001 C CNN
+F 3 "" H 2600 6850 50  0001 C CNN
+	1    2600 6850
 	1    0    0    -1
 $EndComp
@@
 L power:-12V #PWR065
 U 1 1 5DCAAD4A
-P 4400 6650
-F 0 "#PWR065" H 4400 6750 50  0001 C CNN
-F 1 "-12V" H 4415 6823 50  0000 C CNN
-F 2 "" H 4400 6650 50  0001 C CNN
-F 3 "" H 4400 6650 50  0001 C CNN
-	1    4400 6650
-	1    0    0    -1
-$EndComp
-Wire Wire Line
-	3750 7000 4100 7000
+P 2900 7200
+F 0 "#PWR065" H 2900 7300 50  0001 C CNN
+F 1 "-12V" H 2915 7373 50  0000 C CNN
+F 2 "" H 2900 7200 50  0001 C CNN
+F 3 "" H 2900 7200 50  0001 C CNN
+	1    2900 7200
+	-1   0    0    1
+$EndComp
 Wire Wire Line
 	5700 4950 5700 4650
@@
 VIDEO_COMP
 Wire Wire Line
-	4400 6650 4400 6700
-Wire Wire Line
-	3750 6650 3750 6700
-Wire Wire Line
-	4100 7000 4400 7000
-Connection ~ 4100 7000
+	2900 6350 2900 6400
 Wire Wire Line
 	5700 3650 5700 4650
@@
 	5700 4650 6600 4650
 Wire Wire Line
-	3700 950  3700 1000
-Wire Wire Line
-	4400 950  4400 1000
-Wire Wire Line
-	4100 1300 4400 1300
-Connection ~ 4100 1300
+	3100 800  3100 850
 $Comp
 L Device:C C29
@@
 L power:GND #PWR073
 U 1 1 5DCAAD4F
-P 6600 5150
-F 0 "#PWR073" H 6600 4900 50  0001 C CNN
-F 1 "GND" H 6605 4977 50  0000 C CNN
-F 2 "" H 6600 5150 50  0001 C CNN
-F 3 "" H 6600 5150 50  0001 C CNN
-	1    6600 5150
+P 6400 5350
+F 0 "#PWR073" H 6400 5100 50  0001 C CNN
+F 1 "GND" H 6405 5177 50  0000 C CNN
+F 2 "" H 6400 5350 50  0001 C CNN
+F 3 "" H 6400 5350 50  0001 C CNN
+	1    6400 5350
 	1    0    0    -1
 $EndComp
@@
 L power:+12V #PWR061
 U 1 1 5DC9BD5F
-P 3750 6650
-F 0 "#PWR061" H 3750 6500 50  0001 C CNN
-F 1 "+12V" H 3765 6823 50  0000 C CNN
-F 2 "" H 3750 6650 50  0001 C CNN
-F 3 "" H 3750 6650 50  0001 C CNN
-	1    3750 6650
+P 2900 6350
+F 0 "#PWR061" H 2900 6200 50  0001 C CNN
+F 1 "+12V" H 2915 6523 50  0000 C CNN
+F 2 "" H 2900 6350 50  0001 C CNN
+F 3 "" H 2900 6350 50  0001 C CNN
+	1    2900 6350
 	1    0    0    -1
 $EndComp
@@
 L power:GND #PWR075
 U 1 1 5DCAAD32
-P 8600 5000
-F 0 "#PWR075" H 8600 4750 50  0001 C CNN
-F 1 "GND" H 8605 4827 50  0000 C CNN
-F 2 "" H 8600 5000 50  0001 C CNN
-F 3 "" H 8600 5000 50  0001 C CNN
-	1    8600 5000
+P 8600 5200
+F 0 "#PWR075" H 8600 4950 50  0001 C CNN
+F 1 "GND" H 8605 5027 50  0000 C CNN
+F 2 "" H 8600 5200 50  0001 C CNN
+F 3 "" H 8600 5200 50  0001 C CNN
+	1    8600 5200
 	1    0    0    -1
 $EndComp
@@
 L power:GND #PWR074
 U 1 1 5DD06114
-P 8600 2600
-F 0 "#PWR074" H 8600 2350 50  0001 C CNN
-F 1 "GND" H 8605 2427 50  0000 C CNN
-F 2 "" H 8600 2600 50  0001 C CNN
-F 3 "" H 8600 2600 50  0001 C CNN
-	1    8600 2600
+P 8600 2850
+F 0 "#PWR074" H 8600 2600 50  0001 C CNN
+F 1 "GND" H 8605 2677 50  0000 C CNN
+F 2 "" H 8600 2850 50  0001 C CNN
+F 3 "" H 8600 2850 50  0001 C CNN
+	1    8600 2850
 	1    0    0    -1
 $EndComp
@@
 Wire Notes Line
 	10900 4800 9150 4800
+Wire Wire Line
+	2500 3100 2500 3350
+Wire Wire Line
+	6600 2750 6450 2750
+Wire Wire Line
+	6450 2750 6450 2950
+Wire Wire Line
+	6600 5150 6400 5150
+Wire Wire Line
+	6400 5150 6400 5350
+Wire Wire Line
+	8600 5000 8600 5200
+Wire Wire Line
+	8600 2600 8600 2850
+$Comp
+L power:-12V #PWR064
+U 1 1 5DB63B14
+P 3100 1650
+F 0 "#PWR064" H 3100 1750 50  0001 C CNN
+F 1 "-12V" H 3115 1823 50  0000 C CNN
+F 2 "" H 3100 1650 50  0001 C CNN
+F 3 "" H 3100 1650 50  0001 C CNN
+	1    3100 1650
+	-1   0    0    1
+$EndComp
+Wire Wire Line
+	3100 1150 3100 1200
+Wire Wire Line
+	3100 1550 3100 1650
+Wire Wire Line
+	3100 1200 2750 1200
+Wire Wire Line
+	2750 1200 2750 1300
+Connection ~ 3100 1200
+Wire Wire Line
+	3100 1200 3100 1250
+Wire Wire Line
+	2900 6700 2900 6750
+Wire Wire Line
+	2900 6750 2600 6750
+Wire Wire Line
+	2600 6750 2600 6850
+Connection ~ 2900 6750
+Wire Wire Line
+	2900 6750 2900 6800
+Wire Wire Line
+	2900 7100 2900 7200
+Text Notes 700  3600 0    50   ~ 0
+JP7\nSelección de Carga de Entrada R7\n\n
+Text Notes 700  6350 0    50   ~ 0
+JP8\nSelección de Carga de Entrada R8\n\n
+Text Notes 5400 3650 2    50   ~ 0
+JP9\nSelección salida negada\n\n
+Text Notes 5400 6400 2    50   ~ 0
+JP10\nSelección de salida negada\n\n
 $EndSCHEMATC

Commit message: pcb, work in progress
Parts:
- removed C29: 0.1uF-50V, Capacitor_SMD:C_0805_2012Metric, symbol Device:C
- removed J21, J23: Conn_Coaxial, Connector_Coaxial:SMA_Amphenol_901-144_Vertical, symbol Connector:Conn_Coaxial
- removed U24: TLV2772IDR, Package_SO:SOIC-8_3.9x4.9mm_P1.27mm, symbol TLV2772IDR:TLV2772IDR
Other:
- moved on the sheet: TP4
Changed lines of the file:
@@
 L Connector:TestPoint TP4
 U 1 1 5E25996A
-P 5700 5900
-F 0 "TP4" H 5642 5926 50  0000 R CNN
-F 1 "TestPoint" H 5642 6017 50  0000 R CNN
-F 2 "TestPoint:TestPoint_THTPad_1.5x1.5mm_Drill0.7mm" H 5900 5900 50  0001 C CNN
-F 3 "~" H 5900 5900 50  0001 C CNN
-	1    5700 5900
+P 6500 5150
+F 0 "TP4" H 6442 5176 50  0000 R CNN
+F 1 "TestPoint" H 6442 5267 50  0000 R CNN
+F 2 "TestPoint:TestPoint_THTPad_1.5x1.5mm_Drill0.7mm" H 6700 5150 50  0001 C CNN
+F 3 "~" H 6700 5150 50  0001 C CNN
+	1    6500 5150
 	-1   0    0    1
 $EndComp
@@
 $EndComp
 Wire Wire Line
-	5700 4950 5700 4650
-$Comp
-L power:+5V #PWR072
-U 1 1 5DCAAD4B
-P 6600 4050
-F 0 "#PWR072" H 6600 3900 50  0001 C CNN
-F 1 "+5V" H 6615 4223 50  0000 C CNN
-F 2 "" H 6600 4050 50  0001 C CNN
-F 3 "" H 6600 4050 50  0001 C CNN
-	1    6600 4050
-	1    0    0    -1
-$EndComp
-$Comp
-L TLV2772IDR:TLV2772IDR U24
-U 1 1 5DCAAD4C
-P 7300 4650
-F 0 "U24" H 7300 5220 50  0000 C CNN
-F 1 "TLV2772IDR" H 7300 5129 50  0000 C CNN
-F 2 "Package_SO:SOIC-8_3.9x4.9mm_P1.27mm" H 7300 4650 50  0001 L BNN
-F 3 "296-1902-1-ND" H 7300 4650 50  0001 L BNN
-F 4 "Texas Instruments" H 7300 4650 50  0001 L BNN "Campo4"
-F 5 "Dual 2.7-V High Slew Rate Rail-To-Rail Output Operational Amplifier 8-SOIC -40 to 125" H 7300 4650 50  0001 L BNN "Campo5"
-F 6 "TLV2772IDR" H 7300 4650 50  0001 L BNN "Campo6"
-F 7 "https://www.digikey.com/product-detail/en/texas-instruments/TLV2772IDR/296-1902-1-ND/405014?utm_source=snapeda&utm_medium=aggregator&utm_campaign=symbol" H 7300 4650 50  0001 L BNN "Campo7"
-F 8 "SOIC-8 Texas Instruments" H 7300 4650 50  0001 L BNN "Campo8"
-	1    7300 4650
-	1    0    0    -1
-$EndComp
-$Comp
-L Connector:Conn_Coaxial J23
-U 1 1 5DCAAD4D
-P 8700 4350
-F 0 "J23" H 8800 4325 50  0000 L CNN
-F 1 "Conn_Coaxial" H 8800 4234 50  0000 L CNN
-F 2 "Connector_Coaxial:SMA_Amphenol_901-144_Vertical" H 8700 4350 50  0001 C CNN
-F 3 " ~" H 8700 4350 50  0001 C CNN
-	1    8700 4350
-	1    0    0    -1
-$EndComp
-$Comp
-L Connector:Conn_Coaxial J21
-U 1 1 5DCAAD4E
-P 8450 4650
-F 0 "J21" H 8100 4550 50  0000 L CNN
-F 1 "Conn_Coaxial" H 7850 4450 50  0000 L CNN
-F 2 "Connector_Coaxial:SMA_Amphenol_901-144_Vertical" H 8450 4650 50  0001 C CNN
-F 3 " ~" H 8450 4650 50  0001 C CNN
-	1    8450 4650
-	1    0    0    -1
-$EndComp
-Wire Wire Line
-	8000 4450 8100 4450
-Wire Wire Line
-	8000 4550 8100 4550
-Wire Wire Line
-	8100 4550 8100 4650
-Wire Wire Line
-	8000 4650 8100 4650
-Wire Wire Line
-	8000 4350 8100 4350
-Wire Wire Line
-	8100 4350 8100 4450
-Wire Wire Line
-	5700 4950 6600 4950
-$Comp
-L power:GND #PWR069
-U 1 1 5DC9BD35
-P 6450 4400
-F 0 "#PWR069" H 6450 4150 50  0001 C CNN
-F 1 "GND" H 6455 4227 50  0000 C CNN
-F 2 "" H 6450 4400 50  0001 C CNN
-F 3 "" H 6450 4400 50  0001 C CNN
-	1    6450 4400
-	1    0    0    -1
-$EndComp
-Wire Wire Line
-	6600 4050 6600 4100
-Wire Wire Line
-	5700 4950 5700 5900
-Connection ~ 5700 4950
-Wire Wire Line
 	9400 3650 5700 3650
 Text Label 7700 3450 0    50   ~ 0
@@
 	2900 6350 2900 6400
 Wire Wire Line
-	5700 3650 5700 4650
-Connection ~ 5700 4650
-Wire Wire Line
-	5700 4650 6600 4650
-Wire Wire Line
 	3100 800  3100 850
-$Comp
-L Device:C C29
-U 1 1 5DC9BD34
-P 6450 4250
-F 0 "C29" H 6200 4250 50  0000 L CNN
-F 1 "0.1uF-50V" H 6000 4150 50  0000 L CNN
-F 2 "Capacitor_SMD:C_0805_2012Metric" H 6488 4100 50  0001 C CNN
-F 3 "~" H 6450 4250 50  0001 C CNN
-	1    6450 4250
-	1    0    0    -1
-$EndComp
 $Comp
 L Device:C C30
@@
 NoConn ~ 4800 2800
 Wire Wire Line
-	6450 4100 6600 4100
-Connection ~ 6600 4100
-Wire Wire Line
-	6600 4100 6600 4450
-Wire Wire Line
 	4900 2500 4900 2550
 Wire Wire Line
@@
 Wire Wire Line
 	2500 2450 2500 2500
-$Comp
-L power:GND #PWR073
-U 1 1 5DCAAD4F
-P 6400 5350
-F 0 "#PWR073" H 6400 5100 50  0001 C CNN
-F 1 "GND" H 6405 5177 50  0000 C CNN
-F 2 "" H 6400 5350 50  0001 C CNN
-F 3 "" H 6400 5350 50  0001 C CNN
-	1    6400 5350
-	1    0    0    -1
-$EndComp
 $Comp
 L power:+5V #PWR067
@@
 	1    0    0    -1
 $EndComp
-$Comp
-L power:GND #PWR075
-U 1 1 5DCAAD32
-P 8600 5200
-F 0 "#PWR075" H 8600 4950 50  0001 C CNN
-F 1 "GND" H 8605 5027 50  0000 C CNN
-F 2 "" H 8600 5200 50  0001 C CNN
-F 3 "" H 8600 5200 50  0001 C CNN
-	1    8600 5200
-	1    0    0    -1
-$EndComp
 Wire Wire Line
 	5700 3450 9400 3450
@@
 Wire Wire Line
 	10450 4050 10450 4250
-Wire Wire Line
-	8100 4650 8250 4650
-Connection ~ 8100 4650
-Wire Wire Line
-	8100 4350 8500 4350
-Connection ~ 8100 4350
-Wire Wire Line
-	8450 4850 8450 5000
-Wire Wire Line
-	8450 5000 8600 5000
-Wire Wire Line
-	8700 5000 8700 4550
-Wire Wire Line
-	8600 5000 8700 5000
-Connection ~ 8600 5000
 $Comp
 L Connector:Conn_Coaxial J22
@@
 Wire Notes Line
 	5000 3800 3250 3800
-Text Notes 6500 6100 0    50   Italic 0
+Text Notes 6500 4450 0    50   Italic 0
 U2_X: Amplificadores operacionales\nSalidas duplicadas para otros equipos\nTensión de salida: 5V
 Wire Notes Line
-	6450 5800 6450 6150
-Wire Notes Line
-	6450 6150 8200 6150
-Wire Notes Line
-	8200 6150 8200 5800
-Wire Notes Line
-	8200 5800 6450 5800
+	6450 4150 6450 4500
+Wire Notes Line
+	6450 4500 8200 4500
+Wire Notes Line
+	8200 4500 8200 4150
+Wire Notes Line
+	8200 4150 6450 4150
 Text Notes 9200 5100 0    50   Italic 0
 U3_X: Convertidor de Niveles Lógicos\nTensión de señal de entrada 5 V\nTensión de señal de salida 3.3V
@@
 Wire Wire Line
 	6450 2750 6450 2950
-Wire Wire Line
-	6600 5150 6400 5150
-Wire Wire Line
-	6400 5150 6400 5350
-Wire Wire Line
-	8600 5000 8600 5200
 Wire Wire Line
 	8600 2600 8600 2850
@@
 Text Notes 5400 6400 2    50   ~ 0
 JP10\nSelección de salida negada\n\n
+Wire Wire Line
+	5700 3650 5700 4950
+Wire Wire Line
+	5700 4950 6500 4950
+Wire Wire Line
+	6500 4950 6500 5150
+Connection ~ 5700 4950
+Text Label 6000 4950 0    50   ~ 0
+VIDEO_COMP
 $EndSCHEMATC

Commit message: mejorando BOM - work in progress
Parts:
- U13, U14: Número de Parte (Digi-Key) (none) -> 296-47682-1-ND
- U23: Descripción (inglés) (none) -> General Purpose Amplifier 2 Circuit Rail-to-Rail 8-SOIC; Enlace (none) -> https://www.digikey.com/product-detail/en/texas-instruments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; Fabricante (none) -> Texas Instruments; Número de Parte (Digi-Key) (none) -> 296-1902-2-ND; Número de parte (Digi-Key) (none) -> 296-1902-2-ND
- U32: Descripción (inglés) (none) -> Dual-Bit Dual-Supply Bus Transceiver With Configurable Volt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; Enlace (none) -> https://www.digikey.com/product-detail/en/texas-instruments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; Fabricante (none) -> Texas Instruments; Número de Parte (Digi-Key) (none) -> 296-17014-1-ND; Número de parte (Digi-Key) (none) -> 296-17014-1-ND
Changed lines of the file:
@@
 F 6 "296-47682-1-ND" H 4100 2500 50  0001 L BNN "Número de parte (Digi-Key)"
 F 7 "https://www.digikey.com/product-detail/en/texas-instruments/LM361MX-NOPB/296-47682-1-ND/3526971" H 4100 2500 50  0001 L BNN "Enlace"
+F 8 "296-47682-1-ND" H 4100 2500 50  0001 C CNN "Número de Parte (Digi-Key)"
 	1    4100 2500
 	1    0    0    -1
@@
 F 7 "https://www.digikey.com/product-detail/en/texas-instruments/TLV2772IDR/296-1902-1-ND/405014?utm_source=snapeda&utm_medium=aggregator&utm_campaign=symbol" H 7300 2250 50  0001 L BNN "Campo7"
 F 8 "SOIC-8 Texas Instruments" H 7300 2250 50  0001 L BNN "Campo8"
+F 9 "General Purpose Amplifier 2 Circuit Rail-to-Rail 8-SOIC" H 7300 2250 50  0001 C CNN "Descripción (inglés)"
+F 10 "https://www.digikey.com/product-detail/en/texas-instruments/TLV2772IDR/296-1902-2-ND/374332" H 7300 2250 50  0001 C CNN "Enlace"
+F 11 "Texas Instruments" H 7300 2250 50  0001 C CNN "Fabricante"
+F 12 "296-1902-2-ND" H 7300 2250 50  0001 C CNN "Número de Parte (Digi-Key)"
+F 13 "296-1902-2-ND" H 7300 2250 50  0001 C CNN "Número de parte (Digi-Key)"
 	1    7300 2250
 	1    0    0    -1
@@
 F 2 "Package_SO:VSSOP-8_2.4x2.1mm_P0.5mm" H 9850 3000 50  0001 C CNN
 F 3 "http://www.ti.com/lit/ds/symlink/sn74lvc2t45.pdf" H 8900 3000 50  0001 C CNN
+F 4 "Dual-Bit Dual-Supply Bus Transceiver With Configurable Voltage" H 9800 3550 50  0001 C CNN "Descripción (inglés)"
+F 5 "https://www.digikey.com/product-detail/en/texas-instruments/SN74LVC2T45DCUR/296-17014-2-ND/657833" H 9800 3550 50  0001 C CNN "Enlace"
+F 6 "Texas Instruments" H 9800 3550 50  0001 C CNN "Fabricante"
+F 7 "296-17014-1-ND" H 9800 3550 50  0001 C CNN "Número de Parte (Digi-Key)"
+F 8 "296-17014-1-ND" H 9800 3550 50  0001 C CNN "Número de parte (Digi-Key)"
 	1    9800 3550
 	-1   0    0    -1
@@
 F 6 "296-47682-1-ND" H 4100 5200 50  0001 L BNN "Número de parte (Digi-Key)"
 F 7 "https://www.digikey.com/product-detail/en/texas-instruments/LM361MX-NOPB/296-47682-1-ND/3526971" H 4100 5200 50  0001 L BNN "Enlace"
+F 8 "296-47682-1-ND" H 4100 5200 50  0001 C CNN "Número de Parte (Digi-Key)"
 	1    4100 5200
 	1    0    0    -1
